File: Hardware/Qwiic-OpenLog.brd (EAGLE design)
At the start: 38.1 x 38.1 mm, 58 parts, among them J1 MICRO-SD, J10 GATORGATOR_MINI, J2 GATORGATOR_MINI, J3 GATORGATOR_MINI, J4 GATORGATOR_MINI, J5 ISP, J6 GATORGATOR_MINI, J7 GATORGATOR_MINI, J8 GATORGATOR_MINI, J9 GATORGATOR_MINI, Q1 16MHZ, U1 RV-1805, U2 ATMEGA328P

Commit message: finalizing silk and schematic before design review
Parts:
- added U$19, U$20: (no value), buzzard_labels (4):GATOR#LOG3
- added U$21, U$8: (no value), GatorBit_Final_for_Silk#01#png (3):GATORBIT_FINAL_FOR_SILK#01#PNG
- moved R4 0.63 mm to (34.9, 12.1)
- moved R5 0.63 mm to (34.9, 14.0)
Routing:
- net 3.3V: track 126.1 -> 127.0 mm
- net SDA: track 83.5 -> 82.9 mm
- net SCL: track 74.9 -> 75.6 mm
Changed lines of the file:
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@@
 <?xml version="1.0" encoding="utf-8"?>
 <!DOCTYPE eagle SYSTEM "eagle.dtd">
-<eagle version="9.3.1">
+<eagle version="9.1.0">
 <drawing>
 <settings>
@@
 <attribute name="VALUE" x="26.416" y="22.606" size="0.6096" layer="27" font="vector" ratio="20" align="top-center"/>
 </element>
-<element name="R4" library="SparkFun-Resistors" package="0603" value="10k" x="34.29" y="12.065" smashed="yes" rot="R180">
-<attribute name="NAME" x="34.29" y="11.303" size="0.6096" layer="25" font="vector" ratio="20" rot="R180" align="bottom-center"/>
-<attribute name="PROD_ID" value="RES-00824" x="58.42" y="-36.195" size="1.778" layer="27" font="vector" ratio="15" rot="R180" display="off"/>
-<attribute name="VALUE" value="10k" x="36.957" y="11.811" size="0.6096" layer="27" font="vector" ratio="20" rot="R180" align="top-center"/>
-</element>
-<element name="R5" library="SparkFun-Resistors" package="0603" value="10k" x="34.29" y="13.97" smashed="yes" rot="R180">
-<attribute name="NAME" x="34.29" y="13.208" size="0.6096" layer="25" font="vector" ratio="20" rot="R180" align="bottom-center"/>
-<attribute name="PROD_ID" value="RES-00824" x="64.77" y="-30.48" size="1.778" layer="27" font="vector" ratio="15" rot="R180" display="off"/>
-<attribute name="VALUE" value="10k" x="34.417" y="12.7" size="0.6096" layer="27" font="vector" ratio="20" rot="R180" align="top-center"/>
+<element name="R4" library="SparkFun-Resistors" package="0603" value="10k" x="34.925" y="12.065" smashed="yes" rot="R180">
+<attribute name="NAME" x="34.925" y="11.303" size="0.6096" layer="25" font="vector" ratio="20" rot="R180" align="bottom-center"/>
+<attribute name="PROD_ID" value="RES-00824" x="59.055" y="-36.195" size="1.778" layer="27" font="vector" ratio="15" rot="R180" display="off"/>
+<attribute name="VALUE" value="10k" x="37.592" y="11.811" size="0.6096" layer="27" font="vector" ratio="20" rot="R180" align="top-center"/>
+</element>
+<element name="R5" library="SparkFun-Resistors" package="0603" value="10k" x="34.925" y="13.97" smashed="yes" rot="R180">
+<attribute name="NAME" x="34.925" y="13.208" size="0.6096" layer="25" font="vector" ratio="20" rot="R180" align="bottom-center"/>
+<attribute name="PROD_ID" value="RES-00824" x="65.405" y="-30.48" size="1.778" layer="27" font="vector" ratio="15" rot="R180" display="off"/>
+<attribute name="VALUE" value="10k" x="35.052" y="12.7" size="0.6096" layer="27" font="vector" ratio="20" rot="R180" align="top-center"/>
 </element>
 <element name="J5" library="SparkFun-Connectors" package="2X3_TEST_POINTS" value="ISP" x="10.795" y="16.764" smashed="yes" rot="MR270">
@@
 <attribute name="VALUE" x="28.448" y="5.08" size="0.6096" layer="27" font="vector" ratio="20" rot="R270" align="top-center"/>
 </element>
+<element name="U$8" library="GatorBit_Final_for_Silk#01#png (3)" package="GATORBIT_FINAL_FOR_SILK#01#PNG" value="" x="19.05" y="11.43" rot="MR0"/>
+<element name="U$19" library="buzzard_labels (4)" package="GATOR#LOG3" value="" x="23.114" y="14.859" rot="MR0"/>
+<element name="U$20" library="buzzard_labels (4)" package="GATOR#LOG3" value="" x="25.4" y="13.97"/>
+<element name="U$21" library="GatorBit_Final_for_Silk#01#png (3)" package="GATORBIT_FINAL_FOR_SILK#01#PNG" value="" x="29.591" y="11.43"/>
 </elements>
 <signals>
@@
 <via x="16.256" y="30.7848" extent="1-16" drill="0.381"/>
 <contactref element="J6" pad="P$2"/>
-<via x="19.685" y="10.16" extent="1-16" drill="0.35"/>
+<via x="18.542" y="9.652" extent="1-16" drill="0.35"/>
 <via x="21.463" y="15.621" extent="1-16" drill="0.35"/>
 <via x="19.685" y="20.32" extent="1-16" drill="0.35"/>
@@
 <wire x1="25.273" y1="10.668" x2="26.035" y2="11.43" width="0.1524" layer="1"/>
 <wire x1="26.035" y1="11.43" x2="26.035" y2="12.7" width="0.1524" layer="1"/>
-<wire x1="33.44" y1="13.97" x2="33.44" y2="12.954" width="0.1524" layer="1"/>
-<wire x1="33.44" y1="12.954" x2="33.44" y2="12.065" width="0.1524" layer="1"/>
+<wire x1="34.075" y1="13.97" x2="34.075" y2="13.589" width="0.1524" layer="1"/>
+<wire x1="34.075" y1="13.589" x2="34.075" y2="12.065" width="0.1524" layer="1"/>
 <wire x1="31.35" y1="12.935" x2="31.115" y2="12.7" width="0.1524" layer="1"/>
 <wire x1="31.35" y1="16.0274" x2="31.35" y2="12.935" width="0.1524" layer="1"/>
 <wire x1="31.115" y1="12.7" x2="26.035" y2="12.7" width="0.1524" layer="1"/>
 <wire x1="31.35" y1="12.935" x2="33.421" y2="12.935" width="0.1524" layer="1"/>
+<wire x1="33.44" y1="12.954" x2="34.075" y2="13.589" width="0.1524" layer="1"/>
+<contactref element="D2" pad="C"/>
 <wire x1="33.421" y1="12.935" x2="33.44" y2="12.954" width="0.1524" layer="1"/>
-<contactref element="D2" pad="C"/>
 <wire x1="22.2504" y1="20.32" x2="22.645" y2="20.32" width="0" layer="19" extent="1-16"/>
 <wire x1="21.285203125" y1="21.2852" x2="21.2852" y2="21.2852" width="0" layer="19" extent="1-16"/>
@@
 <contactref element="J7" pad="P$2"/>
 <contactref element="J2" pad="P$2"/>
-<wire x1="36.195" y1="12.065" x2="35.14" y2="12.065" width="0.1524" layer="1"/>
 <wire x1="34.29" y1="30.48" x2="34.29" y2="34.544" width="0.1524" layer="1"/>
 <wire x1="36.0426" y1="19.92" x2="37.103" y2="19.92" width="0.1524" layer="1"/>
 <wire x1="37.103" y1="19.92" x2="37.465" y2="19.558" width="0.1524" layer="1"/>
-<wire x1="37.465" y1="19.558" x2="37.465" y2="13.335" width="0.1524" layer="1"/>
-<wire x1="37.465" y1="13.335" x2="36.195" y2="12.065" width="0.1524" layer="1"/>
 <wire x1="37.103" y1="19.92" x2="37.103" y2="27.667" width="0.1524" layer="1"/>
 <wire x1="37.103" y1="27.667" x2="35.56" y2="29.21" width="0.1524" layer="1"/>
@@
 <wire x1="29.21" y1="6.985" x2="29.845" y2="7.62" width="0.1524" layer="1"/>
 <wire x1="29.845" y1="7.62" x2="34.29" y2="7.62" width="0.1524" layer="1"/>
-<wire x1="34.29" y1="7.62" x2="35.56" y2="7.62" width="0.1524" layer="1"/>
-<wire x1="35.56" y1="7.62" x2="36.195" y2="8.255" width="0.1524" layer="1"/>
-<wire x1="36.195" y1="8.255" x2="36.195" y2="12.065" width="0.1524" layer="1"/>
+<wire x1="35.56" y1="7.62" x2="34.29" y2="7.62" width="0.1524" layer="1"/>
 <wire x1="34.29" y1="3.556" x2="34.29" y2="7.62" width="0.1524" layer="1"/>
+<wire x1="37.465" y1="19.558" x2="37.465" y2="12.065" width="0.1524" layer="1"/>
+<wire x1="37.465" y1="12.065" x2="37.465" y2="9.525" width="0.1524" layer="1"/>
+<wire x1="37.465" y1="9.525" x2="35.56" y2="7.62" width="0.1524" layer="1"/>
+<wire x1="35.775" y1="12.065" x2="37.465" y2="12.065" width="0.1524" layer="1"/>
 </signal>
 <signal name="SDA">
@@
 <wire x1="36.068" y1="27.432" x2="33.02" y2="30.48" width="0.1524" layer="1"/>
 <wire x1="37.084" y1="13.589" x2="36.449" y2="12.954" width="0.1524" layer="1"/>
-<wire x1="34.6557125" y1="12.954" x2="34.29" y2="12.5882875" width="0.1524" layer="1"/>
-<wire x1="36.449" y1="12.954" x2="34.6557125" y2="12.954" width="0.1524" layer="1"/>
-<wire x1="34.29" y1="12.5882875" x2="34.29" y2="11.43" width="0.1524" layer="1"/>
-<wire x1="34.29" y1="11.43" x2="31.75" y2="8.89" width="0.1524" layer="1"/>
+<wire x1="35.2907125" y1="12.954" x2="34.925" y2="12.5882875" width="0.1524" layer="1"/>
+<wire x1="36.449" y1="12.954" x2="35.2907125" y2="12.954" width="0.1524" layer="1"/>
+<wire x1="34.925" y1="12.5882875" x2="34.925" y2="11.43" width="0.1524" layer="1"/>
+<wire x1="34.925" y1="11.43" x2="32.385" y2="8.89" width="0.1524" layer="1"/>
 <wire x1="24.13" y1="3.81" x2="24.13" y2="3.556" width="0.1524" layer="1"/>
 <wire x1="37.084" y1="18.923" x2="37.084" y2="13.97" width="0.1524" layer="1"/>
 <wire x1="37.084" y1="13.97" x2="37.084" y2="13.589" width="0.1524" layer="1"/>
-<wire x1="35.14" y1="13.97" x2="37.084" y2="13.97" width="0.1524" layer="1"/>
+<wire x1="35.775" y1="13.97" x2="37.084" y2="13.97" width="0.1524" layer="1"/>
 <contactref element="U1" pad="5"/>
 <wire x1="9.22" y1="25.57" x2="9.22" y2="24.943" width="0.1524" layer="1"/>
@@
 <wire x1="19.05" y1="6.23" x2="19.05" y2="6.985" width="0.1524" layer="1"/>
 <wire x1="20.955" y1="8.89" x2="19.05" y2="6.985" width="0.1524" layer="1"/>
-<wire x1="31.75" y1="8.89" x2="24.13" y2="8.89" width="0.1524" layer="1"/>
+<wire x1="32.385" y1="8.89" x2="24.13" y2="8.89" width="0.1524" layer="1"/>
 <wire x1="24.13" y1="8.89" x2="20.955" y2="8.89" width="0.1524" layer="1"/>
 <wire x1="24.13" y1="3.556" x2="24.13" y2="8.89" width="0.1524" layer="1"/>

Commit message: engineer run of checklist
Parts:
- added Q2: 2.5A/30V/105mΩ, SparkFun-DiscreteSemi:SOT23-3
- added R8: 10k, SparkFun-Resistors:0603
- added U$22: (no value), SparkFun-Aesthetics:ORDERING_INSTRUCTIONS
- moved FID2 6.63 mm to (1.02, 6.99)
- moved FID3 6.63 mm to (1.02, 6.99)
- moved D2 2.36 mm to (10.3, 6.99)
- moved LOGO1 1.27 mm to (19.1, 8.89)
- moved D4 1.27 mm to (19.1, 3.81)
- moved D5 1.27 mm to (29.2, 3.81)
Connections:
- new net N$5: J4.P$2, J9.P$2, Q2.3
- new net N$6: D2.A, Q2.1, R8.2
- net 3.3V: now also Q2.2; no longer J4.P$2, J9.P$2
- net GND: now also R8.1; no longer D2.A
Routing:
- net N$5: track 0.00 -> 44.0 mm, vias 0 -> 1
- net 3.3V: track 127.0 -> 109.3 mm, vias 4 -> 3
- net N$6: track 0.00 -> 3.01 mm
- net SCL: track 75.6 -> 76.8 mm
- net SDA: track 82.9 -> 83.9 mm
- net GND: track 3.12 -> 3.26 mm, vias 11 -> 16
Other:
- board text added: "Black Gloss Soldermask"

Commit message: pre design review for reds
Parts:
- moved LOGO2 1.27 mm to (19.1, 2.54)
Other:
- board text added: "Units in Inches"
Changed lines of the file:
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@@
 <dimension x1="0" y1="38.1" x2="38.1" y2="38.1" x3="19.05" y3="43.18" textsize="1.778" layer="47" dtype="horizontal" unit="inch"/>
 <text x="-7.62" y="-36.83" size="1.778" layer="51" font="vector">Black Gloss Soldermask</text>
+<text x="8.89" y="39.37" size="1.778" layer="47" font="vector">Units in Inches</text>
 </plain>
 <attributes>
@@
 <element name="FID1" library="SparkFun-Aesthetics" package="FIDUCIAL-MICRO" value="FIDUCIALUFIDUCIAL" x="36.83" y="30.48" smashed="yes"/>
 <element name="FID2" library="SparkFun-Aesthetics" package="FIDUCIAL-MICRO" value="FIDUCIALUFIDUCIAL" x="1.016" y="6.985" smashed="yes"/>
-<element name="LOGO2" library="SparkFun-Aesthetics" package="OSHW-LOGO-MINI" value="OSHW-LOGOMINI" x="19.05" y="1.27" smashed="yes" rot="MR0"/>
+<element name="LOGO2" library="SparkFun-Aesthetics" package="OSHW-LOGO-MINI" value="OSHW-LOGOMINI" x="19.05" y="2.54" smashed="yes" rot="MR0"/>
 <element name="FID3" library="SparkFun-Aesthetics" package="FIDUCIAL-MICRO" value="FIDUCIALUFIDUCIAL" x="1.016" y="6.985" smashed="yes" rot="MR180"/>
 <element name="FID4" library="SparkFun-Aesthetics" package="FIDUCIAL-MICRO" value="FIDUCIALUFIDUCIAL" x="36.83" y="30.48" smashed="yes" rot="MR0"/>
