File: Hardware/Qwiic-OpenLog.brd (EAGLE design)
At the start: 38.1 x 38.1 mm, 67 parts, among them J1 MICRO-SD, J10 GATORGATOR_MINI, J2 GATORGATOR_MINI, J3 GATORGATOR_MINI, J4 GATORGATOR_MINI, J5 ISP, J6 GATORGATOR_MINI, J7 GATORGATOR_MINI, J8 GATORGATOR_MINI, J9 GATORGATOR_MINI, Q1 16MHZ, Q2 2.5A/30V/105mΩ, U2 ATMEGA328P, U3 RV-3028

Commit message: centering silk
Parts:
- moved U$24 0.38 mm to (26.3, 15.2)
Changed lines of the file:
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@@
 </element>
 <element name="U$23" library="buzzard_labels" package="GND0" value="" x="6.2484" y="7.874" smashed="yes" rot="MR0"/>
-<element name="U$24" library="buzzard_labels (17)" package="GATOR#LOG0" value="" x="26.67" y="15.24" rot="MR0"/>
+<element name="U$24" library="buzzard_labels (17)" package="GATOR#LOG0" value="" x="26.289" y="15.24" rot="MR0"/>
 <element name="U$19" library="buzzard_labels (18)" package="TIMESTAMP0" value="" x="8.763" y="29.083" rot="R90"/>
 </elements>
