File: Hardware/OpenLog.brd (EAGLE design)
At the start: 38.1 x 25.4 mm, 29 parts, among them J2 ISP, J5 GATORGATOR_MINI, J6 GATORGATOR_MINI, J7 GATORGATOR_MINI, J8 GATORGATOR_MINI, J9 GATORGATOR_MINI, Q1 16MHZ, Q3 2.5A/30V/105mΩ, U1 ATMEGA328P_TQFP, U3 microSD Socket

Commit message: serial changes, pre design review
Parts:
- added U$1, U$2: (no value), buzzard_labels (3):#RST4
- added U$10, U$9: (no value), buzzard_labels (3):TX1
- added U$11: (no value), buzzard_labels (3):GATOR#LOG6
- added U$12: (no value), buzzard_labels (3):GATOR#LOG5
- added U$13: (no value), SparkFun-Aesthetics:SFE_LOGO_NAME_FLAME_.1
- added U$14: (no value), buzzard_labels (4):ST16
- added U$15: (no value), buzzard_labels (4):ST27
- added U$16: (no value), SparkFun-Aesthetics:GATORBIT_FINAL_FOR_SILK#01_#1##JPG
- added U$3, U$4: (no value), buzzard_labels (3):3V32
- added U$5, U$6: (no value), buzzard_labels (3):GND3
- added U$7, U$8: (no value), buzzard_labels (3):RX0
- moved FID4 14.4 mm to (36.8, 24.1)
- moved LOGO2 10.2 mm to (29.2, 12.7)
- moved R2 5.39 mm to (35.6, 15.2), turned to 270 degrees
- moved LOGO1 5.21 mm to (34.2, 23.4)
- moved C2 1.90 mm to (31.8, 19.1)
- moved FID1 1.42 mm to (0.64, 6.35)
- moved FID3 1.42 mm to (0.64, 6.35)
- moved Q1 0.63 mm to (22.3, 10.8)
- moved FID2 0.57 mm to (36.8, 24.1)
Routing:
- net 3.3V: track 69.2 -> 62.0 mm
- net RST: track 29.7 -> 32.7 mm
- net DTR: track 15.6 -> 18.1 mm
Other:
- board text added: "v20"
- board text removed: "0.8mm Thin PCB"
- board text removed: "V15"
