File: Hardware/GatorLog.brd (EAGLE design)
At the start: 38.1 x 25.4 mm, 45 parts, among them J2 ISP, J5 GATORGATOR_MINI, J6 GATORGATOR_MINI, J7 GATORGATOR_MINI, J8 GATORGATOR_MINI, J9 GATORGATOR_MINI, Q1 16MHZ, Q3 2.5A/30V/105mΩ, U1 ATMEGA328P_TQFP, U3 microSD Socket

Commit message: post checklist changes
Parts:
- added U$17: (no value), SparkFun-Aesthetics:ORDERING_INSTRUCTIONS
- C2, C3: device SparkFun-Capacitors:0603-CAP -> SparkFun-Capacitors:0603
- R1: value 1K -> 1k; device SparkFun-Resistors:0603-RES -> SparkFun-Resistors:0603
- R2: value 10K -> 10k; device SparkFun-Resistors:0603-RES -> SparkFun-Resistors:0603
- R6: device SparkFun-Resistors:0603-RES -> SparkFun-Resistors:0603
- moved U$1 4.38 mm to (21.8, 17.4), turned to 0 degrees
- moved U$2 4.32 mm to (26.3, 17.4), turned to 0 degrees
Routing:
- net DTR: track 18.1 -> 17.5 mm
Other:
- board text added: "A. England"
- board text added: "BLACK PCB"
- board text added: "v10"
- board text removed: "N. Seidle"
- board text removed: "Revised by: Patrick Alberts, Pete Lewis"
- board text removed: "v20"
Changed lines of the file:
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@@
 <board>
 <plain>
-<text x="9.316721875" y="-15.367" size="1.778" layer="51" font="vector" ratio="10">N. Seidle</text>
-<text x="-9.51738125" y="-17.92731875" size="1.778" layer="51" font="vector" ratio="10">Revised by: Patrick Alberts, Pete Lewis</text>
-<text x="19.05" y="0.8255" size="1.016" layer="16" font="vector" ratio="20" rot="MR180" align="center">v20</text>
+<text x="9.316721875" y="-15.367" size="1.778" layer="51" font="vector" ratio="10">A. England</text>
+<text x="19.05" y="0.8255" size="1.016" layer="16" font="vector" ratio="20" rot="MR180" align="center">v10</text>
 <wire x1="0" y1="0" x2="38.1" y2="0" width="0.2032" layer="20"/>
 <wire x1="38.1" y1="0" x2="38.1" y2="25.4" width="0.2032" layer="20"/>
@@
 <dimension x1="38.1" y1="0" x2="38.1" y2="25.4" x3="43.18" y3="12.7" textsize="1.778" textratio="15" layer="47" unit="inch"/>
 <dimension x1="38.1" y1="25.4" x2="0" y2="25.4" x3="19.05" y3="26.67" textsize="1.778" layer="47" unit="inch"/>
+<text x="-2.54" y="-31.75" size="1.778" layer="51">BLACK PCB</text>
 </plain>
 <attributes>
@@
 </autorouter>
 <elements>
-<element name="R2" library="SparkFun-Resistors" package="0603-RES" value="10K" x="35.56" y="15.24" smashed="yes" rot="R270">
+<element name="R2" library="SparkFun-Resistors" package="0603" value="10k" x="35.56" y="15.24" smashed="yes" rot="R270">
 <attribute name="NAME" x="36.2585" y="16.129" size="0.4064" layer="25" rot="R270"/>
 <attribute name="PROD_ID" value="RES-00824" x="35.56" y="15.24" size="1.778" layer="27" rot="R270" display="off"/>
-<attribute name="VALUE" value="10K" x="36.1442" y="15.7353" size="0.4064" layer="27" rot="R270"/>
-</element>
-<element name="C3" library="SparkFun-Capacitors" package="0603-CAP" value="0.1uF" x="21.59" y="15.24" smashed="yes" rot="R270">
+<attribute name="VALUE" value="10k" x="36.1442" y="15.7353" size="0.4064" layer="27" rot="R270"/>
+</element>
+<element name="C3" library="SparkFun-Capacitors" package="0603" value="0.1uF" x="21.59" y="15.24" smashed="yes" rot="R270">
 <attribute name="NAME" x="22.2885" y="16.129" size="0.4064" layer="25" rot="R270"/>
-<attribute name="PROD_ID" value="CAP-00810" x="21.59" y="15.24" size="1.778" layer="27" rot="R270" display="off"/>
+<attribute name="PROD_ID" value="CAP-08604" x="21.59" y="15.24" size="1.778" layer="27" rot="R270" display="off"/>
 <attribute name="VALUE" value="0.1uF" x="22.1234" y="15.9639" size="0.4064" layer="27" rot="R270"/>
 </element>
-<element name="R6" library="SparkFun-Resistors" package="0603-RES" value="330" x="17.78" y="10.16" smashed="yes" rot="R270">
+<element name="R6" library="SparkFun-Resistors" package="0603" value="330" x="17.78" y="10.16" smashed="yes" rot="R270">
 <attribute name="NAME" x="17.78" y="12.16" size="1.27" layer="25" rot="R90"/>
 <attribute name="PROD_ID" value="RES-00818" x="17.78" y="10.16" size="1.778" layer="27" rot="R270" display="off"/>
@@
 <attribute name="VALUE" value="16MHZ" x="19.847559375" y="11.09208125" size="0.4064" layer="27"/>
 </element>
-<element name="C2" library="SparkFun-Capacitors" package="0603-CAP" value="0.1uF" x="31.75" y="19.05">
-<attribute name="PROD_ID" value="CAP-00810" x="31.75" y="19.05" size="1.778" layer="27" display="off"/>
+<element name="C2" library="SparkFun-Capacitors" package="0603" value="0.1uF" x="31.75" y="19.05">
+<attribute name="PROD_ID" value="CAP-08604" x="31.75" y="19.05" size="1.778" layer="27" display="off"/>
 <attribute name="VALUE" value="0.1uF" x="31.75" y="19.05" size="1.778" layer="27" display="off"/>
 </element>
@@
 <attribute name="PROD_ID" value="CONN-07820" x="15.875" y="10.16" size="1.778" layer="27" rot="R90" display="off"/>
 </element>
-<element name="R1" library="SparkFun-Resistors" package="0603-RES" value="1K" x="17.78" y="15.24" rot="R270">
+<element name="R1" library="SparkFun-Resistors" package="0603" value="1k" x="17.78" y="15.24" rot="R270">
 <attribute name="PROD_ID" value="RES-07856" x="17.78" y="15.24" size="1.778" layer="27" rot="R270" display="off"/>
-<attribute name="VALUE" value="1K" x="17.78" y="15.24" size="1.778" layer="27" rot="R270" display="off"/>
+<attribute name="VALUE" value="1k" x="17.78" y="15.24" size="1.778" layer="27" rot="R270" display="off"/>
 </element>
 <element name="D1" library="SparkFun-LED" package="LED-0603" value="BLUE" x="19.685" y="15.24" rot="R90">
@@
 </element>
 <element name="J2" library="SparkFun-Connectors" package="2X3_TEST_POINTS" value="ISP" x="11.43" y="21.59" rot="MR90"/>
-<element name="U$1" library="buzzard_labels (3)" package="#RST4" value="" x="26.2255" y="17.399" rot="R180"/>
-<element name="U$2" library="buzzard_labels (3)" package="#RST4" value="" x="21.971" y="17.399" rot="MR180"/>
+<element name="U$1" library="buzzard_labels (3)" package="#RST4" value="" x="21.844" y="17.399"/>
+<element name="U$2" library="buzzard_labels (3)" package="#RST4" value="" x="26.289" y="17.399" rot="MR0"/>
 <element name="U$3" library="buzzard_labels (3)" package="3V32" value="" x="11.557" y="7.874"/>
 <element name="U$4" library="buzzard_labels (3)" package="3V32" value="" x="16.256" y="7.874" rot="MR0"/>
@@
 <element name="U$15" library="buzzard_labels (4)" package="ST27" value="" x="17.4625" y="12.573"/>
 <element name="U$16" library="SparkFun-Aesthetics" package="GATORBIT_FINAL_FOR_SILK#01_#1##JPG" value="" x="8.6995" y="13.1445" rot="MR0"/>
+<element name="U$17" library="SparkFun-Aesthetics" package="ORDERING_INSTRUCTIONS" value="" x="-3.81" y="-20.32"/>
 </elements>
 <signals>
@@
 <wire x1="17.78" y1="12.7" x2="17.78" y2="11.01" width="0.2032" layer="1"/>
 <wire x1="31.75" y1="9.9" x2="31.62" y2="10.03" width="0.2032" layer="1"/>
-<wire x1="31.62" y1="10.03" x2="31.496" y2="10.154" width="0.2032" layer="1"/>
 <wire x1="30.0847125" y1="10.4267" x2="29.8180125" y2="10.16" width="0.2032" layer="1"/>
 <wire x1="31.62" y1="10.03" x2="31.2233" y2="10.4267" width="0.2032" layer="1"/>
@@
 <contactref element="U1" pad="15"/>
 <wire x1="5.021584375" y1="17.4336875" x2="5.08" y2="17.4336875" width="0.2032" layer="1"/>
-<wire x1="5.08" y1="17.4336875" x2="5.4263125" y2="17.4336875" width="0.2032" layer="1"/>
 <wire x1="31.21" y1="8.4074" x2="31.21" y2="7.588" width="0.2032" layer="1"/>
 <wire x1="31.21" y1="7.588" x2="31.115" y2="7.493" width="0.2032" layer="1"/>
@@
 <wire x1="23.996" y1="21.71" x2="24.003" y2="21.717" width="0.2032" layer="1"/>
 <wire x1="24.003" y1="21.717" x2="24.13" y2="21.844" width="0.2032" layer="1"/>
-<wire x1="32.6" y1="19.05" x2="32.6" y2="19.47" width="0.2032" layer="1"/>
-<wire x1="24.13" y1="21.59" x2="24.003" y2="21.717" width="0.2032" layer="1"/>
 <wire x1="32.6" y1="19.05" x2="32.6" y2="22.01" width="0.2032" layer="1"/>
 <wire x1="32.6" y1="22.01" x2="31.75" y2="22.86" width="0.2032" layer="1"/>
@@
 <contactref element="U3" pad="CD1"/>
 <contactref element="U1" pad="25"/>
-<wire x1="32.01" y1="16.9926" x2="32.01" y2="16.1059" width="0.2032" layer="1"/>
-<wire x1="32.01" y1="16.1059" x2="31.76455" y2="15.86045" width="0.2032" layer="1"/>
-<via x="31.76455" y="15.86045" extent="1-16" drill="0.381"/>
+<wire x1="32.01" y1="16.9926" x2="32.01" y2="15.9154" width="0.2032" layer="1"/>
+<wire x1="32.01" y1="15.9154" x2="31.70105" y2="15.60645" width="0.2032" layer="1"/>
+<via x="31.70105" y="15.60645" extent="1-16" drill="0.381"/>
 <via x="25.527" y="17.272" extent="1-16" drill="0.381"/>
-<wire x1="30.353" y1="17.272" x2="25.527" y2="17.272" width="0.2032" layer="16"/>
+<wire x1="29.083" y1="17.272" x2="25.527" y2="17.272" width="0.2032" layer="16"/>
 <wire x1="25.527" y1="17.272" x2="22.098" y2="17.272" width="0.2032" layer="1"/>
 <wire x1="16.002" y1="20.32" x2="15.475" y2="20.847" width="0.2032" layer="1"/>
@@
 <wire x1="22.098" y1="17.272" x2="19.05" y2="20.32" width="0.2032" layer="1"/>
 <wire x1="19.05" y1="20.32" x2="16.002" y2="20.32" width="0.2032" layer="1"/>
-<wire x1="31.76455" y1="15.86045" x2="30.353" y2="17.272" width="0.2032" layer="16"/>
+<wire x1="30.74855" y1="15.60645" x2="29.083" y2="17.272" width="0.2032" layer="16"/>
+<wire x1="31.70105" y1="15.60645" x2="30.74855" y2="15.60645" width="0.2032" layer="16"/>
 </signal>
 <signal name="3.3V">
@@
 <mfgpreviewcolor name="substratecolor" color="0xFF786E46"/>
 </mfgpreviewcolors>
+<errors>
+</errors>
 </board>
 </drawing>
