File: Hardware/GatorLog.sch (EAGLE design)
At the start: 29 parts, among them J2 ISP, J5 GATORGATOR_MINI, J6 GATORGATOR_MINI, J7 GATORGATOR_MINI, J8 GATORGATOR_MINI, J9 GATORGATOR_MINI, Q1 16MHZ, Q3 2.5A/30V/105mΩ, U1 ATMEGA328P_TQFP, U3 microSD Socket

Commit message: post checklist changes
Parts:
- C2, C3: device SparkFun-Capacitors:0.1UF-25V(+80/-20%)(0603) -> SparkFun-Capacitors:0.1UF-0603-25V-5%
- R1: value 1K -> 1k; device SparkFun-Resistors:1KOHM-1/10W-1%(0603) -> SparkFun-Resistors:1KOHM-0603-1/10W-1%
- R2: value 10K -> 10k; device SparkFun-Resistors:10KOHM-1/10W-1%(0603)0603 -> SparkFun-Resistors:10KOHM-0603-1/10W-1%
- R6: device SparkFun-Resistors:330OHM1/10W1%(0603) -> SparkFun-Resistors:330OHM-0603-1/10W-1%
Other:
- note added: "A. England"
- note added: "ATMEGA328 VIN:3.0-3.6V"
- note added: "Connections:"
- note added: "ISP Header:"
- note added: "Original OpenLog by N. Seidle"
- note added: "v10"
- note removed: "0.8mm Thin PCB"
- note removed: "N. Seidle"
- note removed: "Power Circuit:"
- note removed: "Remember, RXI is an input pin into OpenLog."
- note removed: "Revised by: Patrick Alberts, Pete Lewis"
- note removed: "SPI Header:"
- note removed: "Serial Header:"
- note removed: "This board cannot be directly connected to an FTDI Basic."
- note removed: "This board is meant to couple directly to Arduino Pro and Pro Mini."
- note removed: "To connect OpenLog to an FTDI basic, you will need to swap TX and RX lines between boards."
- note removed: "V15"
- moved on the sheet: D2, D4, D5, D6, J2, J5, J6, J7, J8, J9, Q3, R3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
