File: Hardware/Production/Qwiic-OpenLog-Panel.brd (EAGLE design)
At the start: 200.9 x 128.3 mm, 1350 parts, among them J1 MICRO-SD, J10 ISP, J100 ISP, J102 MICRO-SD, J103 SMD, J104 PTH, J105 SMD, J106 ISP, J108 MICRO-SD, J109 SMD, J110 PTH, J111 SMD, J112 ISP, J114 MICRO-SD, J115 SMD, J116 PTH, J117 SMD, J118 ISP, J12 MICRO-SD, J120 MICRO-SD, J121 SMD, J122 PTH, J123 SMD, J124 ISP, J126 MICRO-SD, J127 SMD, J128 PTH, J129 SMD, J13 SMD, J130 ISP, J132 MICRO-SD, J133 SMD, J134 PTH, J135 SMD, J136 ISP, J138 MICRO-SD, J139 SMD, J14 PTH, J140 PTH, J141 SMD, J142 ISP, J144 MICRO-SD, J145 SMD, J146 PTH, J147 SMD, J148 ISP, J15 SMD, J150 MICRO-SD, J151 SMD, J152 PTH, J153 SMD, J154 ISP, J156 MICRO-SD, J157 SMD, J158 PTH, J159 SMD, J16 ISP, J160 ISP, J162 MICRO-SD, J163 SMD, J164 PTH, J165 SMD, J166 ISP, J168 MICRO-SD, J18 MICRO-SD, J19 SMD, J2 SMD, J20 PTH, J21 SMD, J22 ISP, J24 MICRO-SD, J25 SMD, J26 PTH, J27 SMD, J28 ISP, J3 PTH, J30 MICRO-SD, J31 SMD, J32 PTH, J33 SMD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

Commit message: panel
Parts:
- removed ADR, ADR1, ADR10, ADR11, ADR12, ADR13, ADR14, ADR15, ADR16, ADR17, ADR18, ADR19, ADR2, ADR20, ADR21, ADR22, ADR23, ADR24, ADR25, ADR26, ADR27, ADR3, ADR4, ADR5, ADR6, ADR7, ADR8, ADR9: (no value), SparkFun:SJ_2S-NO
- removed C33, C36, C39, C42, C45, C48, C51, C54, C57, C60, C63, C66, C69, C72, C75, C78, C81, C84: 4.7uF, SparkFun-Capacitors:0603
- removed C34, C35, C37, C38, C40, C41, C43, C44, C46, C47, C49, C50, C52, C53, C55, C56, C58, C59, C61, C62, C64, C65, C67, C68, C70, C71, C73, C74, C76, C77, C79, C80, C82, C83: 0.1uF, SparkFun-Capacitors:0603
- removed D41, D43, D45, D47, D49, D51, D53, D55: GREEN, SparkFun-LED:LED-0603
- removed D42, D44, D46, D48, D50, D52, D54, D56: RED, SparkFun-LED:LED-0603
- removed E$4: (no value), SparkFun-Aesthetics:FIDUCIAL-1X2
- removed E$5, E$6: (no value), SparkFun-Retired:FIDUCIAL-1.5X3
- removed FID100, FID101, FID102, FID103, FID104, FID105, FID106, FID107, FID108, FID109, FID110, FID111, FID112, FID33, FID34, FID35, FID36, FID37, FID38, FID39, FID40, FID41, FID42, FID43, FID44, FID45, FID46, FID47, FID48, FID49, FID50, FID51, FID52, FID53, FID54, FID55, FID56, FID57, FID58, FID59, FID60, FID61, FID62, FID63, FID64, FID65, FID66, FID67, FID68, FID69, FID70, FID71, FID72, FID73, FID74, FID75, FID76, FID77, FID78, FID79, FID80, FID81, FID82, FID83, FID84, FID85, FID86, FID87, FID88, FID89, FID90, FID91, FID92, FID93, FID94, FID95, FID96, FID97, FID98, FID99: FIDUCIALUFIDUCIAL, SparkFun-Aesthetics:FIDUCIAL-MICRO
- removed I2C, I2C1, I2C10, I2C11, I2C12, I2C13, I2C14, I2C15, I2C16, I2C17, I2C18, I2C19, I2C2, I2C20, I2C21, I2C22, I2C23, I2C24, I2C25, I2C26, I2C27, I2C3, I2C4, I2C5, I2C6, I2C7, I2C8, I2C9: (no value), SparkFun-Jumpers:SMT-JUMPER_3_2-NC_TRACE_SILK
- removed J100, J106, J112, J118, J124, J130, J136, J142, J148, J154, J160, J166, J82, J88, J94: ISP, SparkFun-Connectors:2X3_TEST_POINTS
- removed J101, J107, J113, J119, J125, J131, J137, J143, J149, J155, J161, J167, J83, J89, J95: (no value), SparkFun-Connectors:1X06_NO_SILK
- removed J102, J108, J114, J120, J126, J132, J138, J144, J150, J156, J162, J168, J84, J90, J96: MICRO-SD, SparkFun-Connectors:MICRO-SD-SOCKET
- removed J103, J105, J109, J111, J115, J117, J121, J123, J127, J129, J133, J135, J139, J141, J145, J147, J151, J153, J157, J159, J163, J165, J81, J85, J87, J91, J93, J97, J99: SMD, SparkFun-Connectors:1X04_1MM_RA
- removed J104, J110, J116, J122, J128, J134, J140, J146, J152, J158, J164, J86, J92, J98: PTH, SparkX:1X04_NO_SILK
- removed JP1, JP10, JP11, JP12, JP13, JP14, JP15, JP16, JP17, JP18, JP19, JP2, JP20, JP21, JP22, JP23, JP24, JP25, JP26, JP27, JP28, JP29, JP3, JP30, JP31, JP32, JP33, JP34, JP35, JP36, JP37, JP38, JP39, JP4, JP40, JP41, JP42, JP43, JP44, JP45, JP46, JP47, JP48, JP49, JP5, JP50, JP51, JP52, JP53, JP54, JP55, JP56, JP6, JP7, JP8, JP9: STAND-OFF, SparkFun:STAND-OFF
- removed LOGO25, LOGO28, LOGO31, LOGO34, LOGO37, LOGO40, LOGO43, LOGO46, LOGO49, LOGO52, LOGO55, LOGO58, LOGO61, LOGO64, LOGO67, LOGO70, LOGO73, LOGO76, LOGO79, LOGO82: OSHW-LOGOMINI, SparkFun-Aesthetics:OSHW-LOGO-MINI
- removed LOGO26, LOGO29, LOGO32, LOGO35, LOGO38, LOGO41, LOGO44, LOGO47, LOGO50, LOGO53, LOGO56, LOGO59, LOGO62, LOGO65, LOGO68, LOGO71, LOGO74, LOGO77, LOGO80, LOGO83: SFE_LOGO_NAME_FLAME.1_INCH, SparkFun-Aesthetics:SFE_LOGO_NAME_FLAME_.1
- removed LOGO27, LOGO30, LOGO33, LOGO36, LOGO39, LOGO42, LOGO45, LOGO48, LOGO51, LOGO54, LOGO57, LOGO60, LOGO63, LOGO66, LOGO69, LOGO72, LOGO75, LOGO78, LOGO81, LOGO84: SFE_LOGO_FLAME.1_INCH, SparkFun-Aesthetics:SFE_LOGO_FLAME_.1
- removed Q17, Q18, Q19, Q20, Q21, Q22, Q23, Q24, Q25, Q26, Q27, Q28: 16MHZ, SparkFun-FreqCtrl:RESONATOR-SMD
- removed R100, R101, R106, R107, R112, R113, R118, R119, R124, R125, R130, R131, R136, R137, R142, R143, R148, R149, R154, R155, R160, R161, R166, R167, R82, R83, R88, R89, R94, R95: 2.2k, SparkFun-Resistors:0603
- removed R102, R103, R108, R109, R114, R115, R120, R121, R126, R127, R132, R133, R138, R139, R144, R145, R150, R151, R156, R157, R162, R163, R168, R84, R85, R90, R91, R96, R97: 10k, SparkFun-Resistors:0603
- removed R104, R110, R116, R122, R128, R134, R140, R146, R152, R158, R164, R86, R92, R98: 330, SparkFun-Resistors:0603
- removed R105, R111, R117, R123, R129, R135, R141, R147, R153, R159, R165, R81, R87, R93, R99: 1k, SparkFun-Resistors:0603
- removed U$185, U$203, U$221, U$239, U$257, U$275, U$293, U$311, U$329, U$347, U$365, U$383, U$401, U$419, U$437, U$455, U$473, U$491: (no value), Labels:PWR-()-03
- removed U$186, U$204, U$222, U$240, U$258, U$276, U$294, U$312, U$330, U$348, U$366, U$384, U$402, U$420, U$438, U$456, U$474, U$492: (no value), buzzard_labels (13):BLK3
- removed U$187, U$205, U$223, U$241, U$259, U$277, U$295, U$313, U$331, U$349, U$367, U$385, U$403, U$421, U$439, U$457, U$475, U$493: (no value), buzzard_labels (13):BOOT5
- removed U$188, U$206, U$224, U$242, U$260, U$278, U$296, U$314, U$332, U$350, U$368, U$386, U$404, U$422, U$440, U$458, U$476, U$494: (no value), buzzard_labels (13):GRN4
- removed U$189, U$207, U$225, U$243, U$261, U$279, U$297, U$315, U$333, U$351, U$369, U$387, U$405, U$423, U$441, U$459, U$477, U$495: (no value), buzzard_labels (13):QWIIC7
- removed U$190, U$195, U$208, U$213, U$226, U$231, U$244, U$249, U$262, U$267, U$280, U$285, U$298, U$303, U$316, U$321, U$334, U$339, U$352, U$357, U$370, U$375, U$388, U$393, U$406, U$411, U$424, U$429, U$442, U$447, U$460, U$465, U$478, U$483, U$496, U$501: (no value), buzzard_labels (13):SCL2
- removed U$191, U$194, U$209, U$212, U$227, U$230, U$245, U$248, U$263, U$266, U$281, U$284, U$299, U$302, U$317, U$320, U$335, U$338, U$353, U$356, U$371, U$374, U$389, U$392, U$407, U$410, U$425, U$428, U$443, U$446, U$461, U$464, U$479, U$482, U$497, U$500: (no value), buzzard_labels (13):SDA1
- removed U$192, U$210, U$228, U$246, U$264, U$282, U$300, U$318, U$336, U$354, U$372, U$390, U$408, U$426, U$444, U$462, U$480, U$498: (no value), buzzard_labels (13):STAT0
- removed U$193, U$211, U$229, U$247, U$265, U$283, U$301, U$319, U$337, U$355, U$373, U$391, U$409, U$427, U$445, U$463, U$481, U$499: (no value), buzzard_labels (14):OPENLOG0
- removed U$196, U$214, U$232, U$250, U$268, U$286, U$304, U$322, U$340, U$358, U$376, U$394, U$412, U$430, U$448, U$466, U$484, U$502: (no value), buzzard_labels (16):3V30
- removed U$197, U$215, U$233, U$251, U$269, U$287, U$305, U$323, U$341, U$359, U$377, U$395, U$413, U$431, U$449, U$467, U$485, U$503: (no value), buzzard_labels (16):GND1
- removed U$198, U$216, U$234, U$252, U$270, U$288, U$306, U$324, U$342, U$360, U$378, U$396, U$414, U$432, U$450, U$468, U$486, U$504: (no value), Labels:QWIIC-LOGO-SMALL
- removed U$199, U$217, U$235, U$253, U$271, U$289, U$307, U$325, U$343, U$361, U$379, U$397, U$415, U$433, U$451, U$469, U$487: (no value), Labels:3V3-03
- removed U$200, U$218, U$236, U$254, U$272, U$290, U$308, U$326, U$344, U$362, U$380, U$398, U$416, U$434, U$452, U$470, U$488: (no value), Labels:GND-03
- removed U$201, U$219, U$237, U$255, U$273, U$291, U$309, U$327, U$345, U$363, U$381, U$399, U$417, U$435, U$453, U$471, U$489: (no value), Labels:ADR-()-03
- removed U$202, U$220, U$238, U$256, U$274, U$292, U$310, U$328, U$346, U$364, U$382, U$400, U$418, U$436, U$454, U$472, U$490: (no value), Labels:I_SUPER2_C-()-03
- removed U17, U18, U19, U20, U21, U22, U23, U24, U25, U26, U27, U28: ATMEGA328P, SparkFun-IC-Microcontroller:TQFP32-08
- added BT1, BT2, BT3, BT4, BT5, BT6, BT7, BT8: ML414H_IV01E_BATTERY, SparkFun-Batteries:ML414H_IV01E
- added S1, S2, S3, S4, S5, S6, S7, S8: (no value), SparkFun-Switches:TACTILE_SWITCH_SMD_5.2MM
- C10, C14, C22, C26: value 0.1uF -> 4.7uF
- C12, C15, C21, C24, C27, C9: value 4.7uF -> 0.1uF
- D10, D14, D18, D20, D24, D28, D30, D34, D38, D4, D40, D8: value RED -> 3.6V; device SparkFun-LED:LED-0603 -> SparkFun-DiscreteSemi:SOD-323
- D13, D15, D19, D2, D23, D25, D29, D33, D35, D39, D5, D9: value GREEN -> 3.6V; device SparkFun-LED:LED-0603 -> SparkFun-DiscreteSemi:SOD-323
- D16, D26, D36, D6: value RED -> GREEN
- D17, D27, D37, D7: value GREEN -> RED
- E$3: device SparkFun-Aesthetics:FIDUCIAL-1X2 -> SparkFun-Retired:FIDUCIAL-1.5X3
- J10, J16, J28, J34, J40, J46, J58, J64, J70, J76: value ISP -> GATORGATOR_MINI; device SparkFun-Connectors:2X3_TEST_POINTS -> SparkFun-Connectors:GATOR_MINI
- J11, J41, J71: value (none) -> ISP; device SparkFun-Connectors:1X06_NO_SILK -> SparkFun-Connectors:2X3_TEST_POINTS
- J13, J15, J19, J2, J25, J27, J33, J37, J39, J4, J43, J45, J49, J55, J57, J63, J67, J69, J7, J73, J75, J79, J9: value SMD -> GATORGATOR_MINI; device SparkFun-Connectors:1X04_1MM_RA -> SparkFun-Connectors:GATOR_MINI
- J14, J20, J26, J3, J38, J44, J50, J56, J68, J74, J8, J80: value PTH -> GATORGATOR_MINI; device SparkX:1X04_NO_SILK -> SparkFun-Connectors:GATOR_MINI
- J17, J23, J29, J35, J47, J53, J59, J6, J65, J77: value (none) -> GATORGATOR_MINI; device SparkFun-Connectors:1X06_NO_SILK -> SparkFun-Connectors:GATOR_MINI
- J18, J24, J30, J36, J48, J54, J60, J66, J78: value MICRO-SD -> GATORGATOR_MINI; device SparkFun-Connectors:MICRO-SD-SOCKET -> SparkFun-Connectors:GATOR_MINI
- J21, J31, J51, J61: value SMD -> ISP; device SparkFun-Connectors:1X04_1MM_RA -> SparkFun-Connectors:2X3_TEST_POINTS
- J22, J52: value ISP -> MICRO-SD; device SparkFun-Connectors:2X3_TEST_POINTS -> SparkFun-Connectors:MICRO-SD-SOCKET
- J32, J62: value PTH -> MICRO-SD; device SparkX:1X04_NO_SILK -> SparkFun-Connectors:MICRO-SD-SOCKET
- Q10, Q12, Q14, Q16, Q2, Q4, Q6, Q8: value 16MHZ -> 2.5A/30V/105mΩ; device SparkFun-FreqCtrl:RESONATOR-SMD -> SparkFun-DiscreteSemi:SOT23-3
- R10, R11, R16, R17, R29, R34, R35, R4, R40, R41, R46, R47, R5, R59, R64, R65, R70, R71, R76, R77: value 2.2k -> 10k
- R12, R42, R72: value 10k -> 330
- R13, R43, R73: value 10k -> 1k
- R14, R20, R26, R44, R50, R56, R74, R8, R80: value 330 -> 10k
- R15, R21, R27, R39, R45, R51, R57, R69, R75, R9: value 1k -> 10k
- R18, R48, R7, R78: value 10k -> 470
- R22, R52: value 2.2k -> 330
- R23, R53: value 2.2k -> 1k
- R28, R58: value 2.2k -> 470
- R38, R68: value 330 -> 470
- U$1, U$127: device Labels:3V3-03 -> buzzard_labels:3V33
- U$10, U$96: device buzzard_labels (13):BLK3 -> buzzard_labels:GND0
- U$100, U$123: device buzzard_labels (13):SCL2 -> buzzard_labels:SCL2
- U$101, U$13, U$16, U$29, U$32: device buzzard_labels (13):SDA1 -> buzzard_labels:SDA1
- U$102: device buzzard_labels (13):STAT0 -> buzzard_labels:GND0
- U$103, U$67: device buzzard_labels (14):OPENLOG0 -> buzzard_labels:GND0
- U$104, U$173, U$176: device buzzard_labels (13):SDA1 -> buzzard_labels:3V33
- U$105, U$154, U$177, U$82: device buzzard_labels (13):SCL2 -> buzzard_labels:SDA1
- U$106, U$178, U$6: device buzzard_labels (16):3V30 -> buzzard_labels:SCL2
- U$107, U$143, U$35: device buzzard_labels (16):GND1 -> buzzard_labels:3V33
- U$108, U$144, U$36: device Labels:QWIIC-LOGO-SMALL -> buzzard_labels:SDA1
- U$109, U$145, U$37: device Labels:3V3-03 -> buzzard_labels:SCL2
- U$11, U$79: device buzzard_labels (13):BOOT5 -> buzzard_labels:GND0
- U$110: device Labels:GND-03 -> GatorBit_Final_for_Silk#01#png (3):GATORBIT_FINAL_FOR_SILK#01#PNG
- U$111: device Labels:ADR-()-03 -> buzzard_labels (4):GATOR#LOG3
- U$112, U$8: device Labels:I_SUPER2_C-()-03 -> GatorBit_Final_for_Silk#01#png (3):GATORBIT_FINAL_FOR_SILK#01#PNG
- U$113, U$149, U$23: device Labels:PWR-()-03 -> buzzard_labels:GND0
- U$114, U$24: device buzzard_labels (13):BLK3 -> buzzard_labels (17):GATOR#LOG0
- U$115: device buzzard_labels (13):BOOT5 -> buzzard_labels (18):TIMESTAMP0
- U$116: device buzzard_labels (13):GRN4 -> Labels:PWR-()-03
- U$117: device buzzard_labels (13):QWIIC7 -> buzzard_labels (13):STAT0
- U$118, U$141, U$15, U$28, U$51: device buzzard_labels (13):SCL2 -> buzzard_labels:3V33
- U$119, U$50: device buzzard_labels (13):SDA1 -> buzzard_labels:GND0
- U$12, U$26: device buzzard_labels (13):GRN4 -> buzzard_labels:3V33
- U$120, U$84: device buzzard_labels (13):STAT0 -> buzzard_labels:3V33
- U$121, U$85: device buzzard_labels (14):OPENLOG0 -> buzzard_labels:SDA1
- U$122, U$155, U$83, U$86: device buzzard_labels (13):SDA1 -> buzzard_labels:SCL2
- U$124, U$52: device buzzard_labels (16):3V30 -> buzzard_labels:SDA1
- U$125: device buzzard_labels (16):GND1 -> buzzard_labels:GND0
- U$126, U$90: device Labels:QWIIC-LOGO-SMALL -> buzzard_labels:GND0
- U$128: device Labels:GND-03 -> buzzard_labels:SDA1
- U$129: device Labels:ADR-()-03 -> buzzard_labels:SCL2
- U$130, U$166, U$58: device Labels:I_SUPER2_C-()-03 -> buzzard_labels:3V33
- U$131, U$167, U$59: device Labels:PWR-()-03 -> buzzard_labels:SDA1
- U$132, U$168, U$60: device buzzard_labels (13):BLK3 -> buzzard_labels:SCL2
- U$133, U$43: device buzzard_labels (13):BOOT5 -> GatorBit_Final_for_Silk#01#png (3):GATORBIT_FINAL_FOR_SILK#01#PNG
- U$134: device buzzard_labels (13):GRN4 -> buzzard_labels (4):GATOR#LOG3
- U$135: device buzzard_labels (13):QWIIC7 -> GatorBit_Final_for_Silk#01#png (3):GATORBIT_FINAL_FOR_SILK#01#PNG
- U$136, U$159, U$172, U$33: device buzzard_labels (13):SCL2 -> buzzard_labels:GND0
- U$137, U$68: device buzzard_labels (13):SDA1 -> buzzard_labels (17):GATOR#LOG0
- U$138: device buzzard_labels (13):STAT0 -> buzzard_labels (18):TIMESTAMP0
- U$139: device buzzard_labels (14):OPENLOG0 -> Labels:PWR-()-03
- U$14, U$63, U$99: device buzzard_labels (13):QWIIC7 -> buzzard_labels:SCL2
- U$140: device buzzard_labels (13):SDA1 -> buzzard_labels (13):STAT0
- U$142, U$34: device buzzard_labels (16):3V30 -> buzzard_labels:GND0
- U$146, U$5: device Labels:GND-03 -> buzzard_labels:SCL2
- U$147, U$39, U$7, U$75: device Labels:ADR-()-03 -> buzzard_labels:SDA1
- U$148: device Labels:I_SUPER2_C-()-03 -> buzzard_labels:GND0
- U$150: device buzzard_labels (13):BLK3 -> buzzard_labels:3V33
- U$151: device buzzard_labels (13):BOOT5 -> buzzard_labels:SDA1
- U$152: device buzzard_labels (13):GRN4 -> buzzard_labels:SCL2
- U$153, U$81: device buzzard_labels (13):QWIIC7 -> buzzard_labels:3V33
- U$156, U$66: device buzzard_labels (13):STAT0 -> GatorBit_Final_for_Silk#01#png (3):GATORBIT_FINAL_FOR_SILK#01#PNG
- U$157: device buzzard_labels (14):OPENLOG0 -> buzzard_labels (4):GATOR#LOG3
- U$158: device buzzard_labels (13):SDA1 -> GatorBit_Final_for_Silk#01#png (3):GATORBIT_FINAL_FOR_SILK#01#PNG
- U$160: device buzzard_labels (16):3V30 -> buzzard_labels (17):GATOR#LOG0
- U$161: device buzzard_labels (16):GND1 -> buzzard_labels (18):TIMESTAMP0
- U$162: device Labels:QWIIC-LOGO-SMALL -> Labels:PWR-()-03
- U$163: device Labels:3V3-03 -> buzzard_labels (13):STAT0
- U$164, U$38, U$74: device Labels:GND-03 -> buzzard_labels:3V33
- U$165, U$57: device Labels:ADR-()-03 -> buzzard_labels:GND0
- U$169: device buzzard_labels (13):BOOT5 -> buzzard_labels:SCL2
- U$170, U$62, U$98: device buzzard_labels (13):GRN4 -> buzzard_labels:SDA1
- U$171, U$27: device buzzard_labels (13):QWIIC7 -> buzzard_labels:GND0
- U$174: device buzzard_labels (13):STAT0 -> buzzard_labels:SDA1
- U$175, U$18, U$31: device buzzard_labels (14):OPENLOG0 -> buzzard_labels:SCL2
- U$179, U$89: device buzzard_labels (16):GND1 -> GatorBit_Final_for_Silk#01#png (3):GATORBIT_FINAL_FOR_SILK#01#PNG
- U$180: device Labels:QWIIC-LOGO-SMALL -> buzzard_labels (4):GATOR#LOG3
- U$181: device Labels:3V3-03 -> GatorBit_Final_for_Silk#01#png (3):GATORBIT_FINAL_FOR_SILK#01#PNG
- U$182, U$2, U$56: device Labels:GND-03 -> buzzard_labels:GND0
- U$183: device Labels:ADR-()-03 -> buzzard_labels (17):GATOR#LOG0
- U$184: device Labels:I_SUPER2_C-()-03 -> buzzard_labels (18):TIMESTAMP0
- U$19, U$46, U$69: device buzzard_labels (13):SCL2 -> buzzard_labels (18):TIMESTAMP0
- U$20: device buzzard_labels (16):GND1 -> buzzard_labels (4):GATOR#LOG3
- U$21: device Labels:ADR-()-03 -> GatorBit_Final_for_Silk#01#png (3):GATORBIT_FINAL_FOR_SILK#01#PNG
- U$22: device Labels:I_SUPER2_C-()-03 -> Labels:PWR-()-03
- U$25: device buzzard_labels (13):BOOT5 -> buzzard_labels (13):STAT0
- U$3, U$72: device Labels:QWIIC-LOGO-SMALL -> buzzard_labels:3V33
- U$30: device buzzard_labels (13):STAT0 -> buzzard_labels:SCL2
- U$4, U$55: device Labels:3V3-03 -> buzzard_labels:SDA1
- U$40, U$76: device Labels:I_SUPER2_C-()-03 -> buzzard_labels:SCL2
- U$41: device Labels:PWR-()-03 -> GatorBit_Final_for_Silk#01#png (3):GATORBIT_FINAL_FOR_SILK#01#PNG
- U$42: device buzzard_labels (13):BLK3 -> buzzard_labels (4):GATOR#LOG3
- U$44, U$80: device buzzard_labels (13):GRN4 -> buzzard_labels:GND0
- U$45: device buzzard_labels (13):QWIIC7 -> buzzard_labels (17):GATOR#LOG0
- U$47: device buzzard_labels (13):SDA1 -> Labels:PWR-()-03
- U$49: device buzzard_labels (14):OPENLOG0 -> buzzard_labels:3V33
- U$53: device buzzard_labels (16):GND1 -> buzzard_labels:SCL2
- U$54: device Labels:QWIIC-LOGO-SMALL -> buzzard_labels:SCL2
- U$61, U$97: device buzzard_labels (13):BOOT5 -> buzzard_labels:3V33
- U$64, U$87: device buzzard_labels (13):SCL2 -> GatorBit_Final_for_Silk#01#png (3):GATORBIT_FINAL_FOR_SILK#01#PNG
- U$65: device buzzard_labels (13):SDA1 -> buzzard_labels (4):GATOR#LOG3
- U$70: device buzzard_labels (16):3V30 -> Labels:PWR-()-03
- U$71: device buzzard_labels (16):GND1 -> buzzard_labels (13):STAT0
- U$73: device Labels:3V3-03 -> buzzard_labels:GND0
- U$77: device Labels:PWR-()-03 -> buzzard_labels:SCL2
- U$78: device buzzard_labels (13):BLK3 -> buzzard_labels:SDA1
- U$88: device buzzard_labels (16):3V30 -> buzzard_labels (4):GATOR#LOG3
- U$91: device Labels:3V3-03 -> buzzard_labels (17):GATOR#LOG0
- U$92: device Labels:GND-03 -> buzzard_labels (18):TIMESTAMP0
- U$93: device Labels:ADR-()-03 -> Labels:PWR-()-03
- U$94: device Labels:I_SUPER2_C-()-03 -> buzzard_labels (13):STAT0
- U$95: device Labels:PWR-()-03 -> buzzard_labels:3V33
- U10, U12, U14, U16, U3, U4, U6, U8: value ATMEGA328P -> RV-3028; device SparkFun-IC-Microcontroller:TQFP32-08 -> SparkFun-Clocks:RV-3028
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Connections:
- removed net 3.3V10: C31.2, C33.1, I2C10.2, J61.2, J62.2, J63.2, J64.2, J65.3, J66.VCC, R61.2, R66.2, U11.18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
- removed net 3.3V11: C34.2, C36.1, I2C11.2, J67.2, J68.2, J69.2, J70.2, J71.3, J72.VCC, R67.2, R72.2, U12.18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
- removed net 3.3V12: C37.2, C39.1, I2C12.2, J73.2, J74.2, J75.2, J76.2, J77.3, J78.VCC, R73.2, R78.2, U13.18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
- removed net 3.3V13: C40.2, C42.1, I2C13.2, J79.2, J80.2, J81.2, J82.2, J83.3, J84.VCC, R79.2, R84.2, U14.18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
- removed net 3.3V14: C43.2, C45.1, I2C14.2, J85.2, J86.2, J87.2, J88.2, J89.3, J90.VCC, R85.2, R90.2, U15.18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
- removed net 3.3V15: C46.2, C48.1, I2C15.2, J91.2, J92.2, J93.2, J94.2, J95.3, J96.VCC, R91.2, R96.2, U16.18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
- removed net 3.3V16: C49.2, C51.1, I2C16.2, J100.2, J101.3, J102.VCC, J97.2, J98.2, J99.2, R102.2, R97.2, U17.18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
- removed net 3.3V17: C52.2, C54.1, I2C17.2, J103.2, J104.2, J105.2, J106.2, J107.3, J108.VCC, R103.2, R108.2, U18.18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
- removed net 3.3V18: C55.2, C57.1, I2C18.2, J109.2, J110.2, J111.2, J112.2, J113.3, J114.VCC, R109.2, R114.2, U19.18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
- removed net 3.3V19: C58.2, C60.1, I2C19.2, J115.2, J116.2, J117.2, J118.2, J119.3, J120.VCC, R115.2, R120.2, U20.18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
- removed net 3.3V20: C61.2, C63.1, I2C20.2, J121.2, J122.2, J123.2, J124.2, J125.3, J126.VCC, R121.2, R126.2, U21.18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
- removed net 3.3V21: C64.2, C66.1, I2C21.2, J127.2, J128.2, J129.2, J130.2, J131.3, J132.VCC, R127.2, R132.2, U22.18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
- removed net 3.3V22: C67.2, C69.1, I2C22.2, J133.2, J134.2, J135.2, J136.2, J137.3, J138.VCC, R133.2, R138.2, U23.18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
- removed net 3.3V23: C70.2, C72.1, I2C23.2, J139.2, J140.2, J141.2, J142.2, J143.3, J144.VCC, R139.2, R144.2, U24.18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
- removed net 3.3V24: C73.2, C75.1, I2C24.2, J145.2, J146.2, J147.2, J148.2, J149.3, J150.VCC, R145.2, R150.2, U25.18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
- removed net 3.3V25: C76.2, C78.1, I2C25.2, J151.2, J152.2, J153.2, J154.2, J155.3, J156.VCC, R151.2, R156.2, U26.18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
- removed net 3.3V26: C79.2, C81.1, I2C26.2, J157.2, J158.2, J159.2, J160.2, J161.3, J162.VCC, R157.2, R162.2, U27.18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
- removed net 3.3V27: C82.2, C84.1, I2C27.2, J163.2, J164.2, J165.2, J166.2, J167.3, J168.VCC, R163.2, R168.2, U28.18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
- removed net 3.3V8: C25.2, C27.1, I2C8.2, J49.2, J50.2, J51.2, J52.2, J53.3, J54.VCC, R49.2, R54.2, U9.18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
- removed net 3.3V9: C28.2, C30.1, I2C9.2, J55.2, J56.2, J57.2, J58.2, J59.3, J60.VCC, R55.2, R60.2, U10.18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
- removed net ADDR10: ADR10.2, U11.1
- removed net ADDR11: ADR11.2, U12.1
- removed net ADDR12: ADR12.2, U13.1
- removed net ADDR13: ADR13.2, U14.1
- removed net ADDR14: ADR14.2, U15.1
- removed net ADDR15: ADR15.2, U16.1
- removed net ADDR16: ADR16.2, U17.1
- removed net ADDR17: ADR17.2, U18.1
- removed net ADDR18: ADR18.2, U19.1
- removed net ADDR19: ADR19.2, U20.1
- removed net ADDR20: ADR20.2, U21.1
- removed net ADDR21: ADR21.2, U22.1
- removed net ADDR22: ADR22.2, U23.1
- removed net ADDR23: ADR23.2, U24.1
- removed net ADDR24: ADR24.2, U25.1
- removed net ADDR25: ADR25.2, U26.1
- removed net ADDR26: ADR26.2, U27.1
- removed net ADDR27: ADR27.2, U28.1
- removed net ADDR8: ADR8.2, U9.1
- removed net ADDR9: ADR9.2, U10.1
- removed net CS10: J66.CS, R66.1, U11.14
- removed net CS11: J72.CS, R72.1, U12.14
- removed net CS12: J78.CS, R78.1, U13.14
- removed net CS13: J84.CS, R84.1, U14.14
- removed net CS14: J90.CS, R90.1, U15.14
- removed net CS15: J96.CS, R96.1, U16.14
- removed net CS16: J102.CS, R102.1, U17.14
- removed net CS17: J108.CS, R108.1, U18.14
- removed net CS18: J114.CS, R114.1, U19.14
- removed net CS19: J120.CS, R120.1, U20.14
- removed net CS20: J126.CS, R126.1, U21.14
- removed net CS21: J132.CS, R132.1, U22.14
- removed net CS22: J138.CS, R138.1, U23.14
- removed net CS23: J144.CS, R144.1, U24.14
- removed net CS24: J150.CS, R150.1, U25.14
- removed net CS25: J156.CS, R156.1, U26.14
- removed net CS26: J162.CS, R162.1, U27.14
- removed net CS27: J168.CS, R168.1, U28.14
- removed net CS8: J54.CS, R54.1, U9.14
- removed net CS9: J60.CS, R60.1, U10.14
- removed net DTR: C2.2, J6.6
- removed net DTR1: C5.2, J11.6
- removed net DTR10: C32.2, J65.6
- removed net DTR11: C35.2, J71.6
- removed net DTR12: C38.2, J77.6
- removed net DTR13: C41.2, J83.6
- removed net DTR14: C44.2, J89.6
- removed net DTR15: C47.2, J95.6
- removed net DTR16: C50.2, J101.6
- removed net DTR17: C53.2, J107.6
- removed net DTR18: C56.2, J113.6
- removed net DTR19: C59.2, J119.6
- removed net DTR2: C8.2, J17.6
- removed net DTR20: C62.2, J125.6
- removed net DTR21: C65.2, J131.6
- removed net DTR22: C68.2, J137.6
- removed net DTR23: C71.2, J143.6
- removed net DTR24: C74.2, J149.6
- removed net DTR25: C77.2, J155.6
- removed net DTR26: C80.2, J161.6
- removed net DTR27: C83.2, J167.6
- removed net DTR3: C11.2, J23.6
- removed net DTR4: C14.2, J29.6
- removed net DTR5: C17.2, J35.6
- removed net DTR6: C20.2, J41.6
- removed net DTR7: C23.2, J47.6
- removed net DTR8: C26.2, J53.6
- removed net DTR9: C29.2, J59.6
- removed net GND10: ADR10.1, C31.1, C33.2, D21.C, D22.C, J61.1, J62.1, J63.1, J64.6, J65.1, J65.2, J66.GND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
- removed net GND11: ADR11.1, C34.1, C36.2, D23.C, D24.C, J67.1, J68.1, J69.1, J70.6, J71.1, J71.2, J72.GND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
- removed net GND12: ADR12.1, C37.1, C39.2, D25.C, D26.C, J73.1, J74.1, J75.1, J76.6, J77.1, J77.2, J78.GND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
- removed net GND13: ADR13.1, C40.1, C42.2, D27.C, D28.C, J79.1, J80.1, J81.1, J82.6, J83.1, J83.2, J84.GND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
- removed net GND14: ADR14.1, C43.1, C45.2, D29.C, D30.C, J85.1, J86.1, J87.1, J88.6, J89.1, J89.2, J90.GND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
- removed net GND15: ADR15.1, C46.1, C48.2, D31.C, D32.C, J91.1, J92.1, J93.1, J94.6, J95.1, J95.2, J96.GND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
- removed net GND16: ADR16.1, C49.1, C51.2, D33.C, D34.C, J100.6, J101.1, J101.2, J102.GND, J97.1, J98.1, J99.1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
- removed net GND17: ADR17.1, C52.1, C54.2, D35.C, D36.C, J103.1, J104.1, J105.1, J106.6, J107.1, J107.2, J108.GND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
- removed net GND18: ADR18.1, C55.1, C57.2, D37.C, D38.C, J109.1, J110.1, J111.1, J112.6, J113.1, J113.2, J114.GND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
- removed net GND19: ADR19.1, C58.1, C60.2, D39.C, D40.C, J115.1, J116.1, J117.1, J118.6, J119.1, J119.2, J120.GND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
- removed net GND20: ADR20.1, C61.1, C63.2, D41.C, D42.C, J121.1, J122.1, J123.1, J124.6, J125.1, J125.2, J126.GND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
- removed net GND21: ADR21.1, C64.1, C66.2, D43.C, D44.C, J127.1, J128.1, J129.1, J130.6, J131.1, J131.2, J132.GND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
- removed net GND22: ADR22.1, C67.1, C69.2, D45.C, D46.C, J133.1, J134.1, J135.1, J136.6, J137.1, J137.2, J138.GND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
- removed net GND23: ADR23.1, C70.1, C72.2, D47.C, D48.C, J139.1, J140.1, J141.1, J142.6, J143.1, J143.2, J144.GND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
- removed net GND24: ADR24.1, C73.1, C75.2, D49.C, D50.C, J145.1, J146.1, J147.1, J148.6, J149.1, J149.2, J150.GND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
- removed net GND25: ADR25.1, C76.1, C78.2, D51.C, D52.C, J151.1, J152.1, J153.1, J154.6, J155.1, J155.2, J156.GND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
- removed net GND26: ADR26.1, C79.1, C81.2, D53.C, D54.C, J157.1, J158.1, J159.1, J160.6, J161.1, J161.2, J162.GND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
- removed net GND27: ADR27.1, C82.1, C84.2, D55.C, D56.C, J163.1, J164.1, J165.1, J166.6, J167.1, J167.2, J168.GND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
- removed net GND8: ADR8.1, C25.1, C27.2, D17.C, D18.C, J49.1, J50.1, J51.1, J52.6, J53.1, J53.2, J54.GND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
- removed net GND9: ADR9.1, C28.1, C30.2, D19.C, D20.C, J55.1, J56.1, J57.1, J58.6, J59.1, J59.2, J60.GND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
- removed net MISO10: J64.1, J66.DO, U11.16
- removed net MISO11: J70.1, J72.DO, U12.16
- removed net MISO12: J76.1, J78.DO, U13.16
- removed net MISO13: J82.1, J84.DO, U14.16
- removed net MISO14: J88.1, J90.DO, U15.16
- removed net MISO15: J94.1, J96.DO, U16.16
- removed net MISO16: J100.1, J102.DO, U17.16
- removed net MISO17: J106.1, J108.DO, U18.16
- removed net MISO18: J112.1, J114.DO, U19.16
- removed net MISO19: J118.1, J120.DO, U20.16
- removed net MISO20: J124.1, J126.DO, U21.16
- removed net MISO21: J130.1, J132.DO, U22.16
- removed net MISO22: J136.1, J138.DO, U23.16
- removed net MISO23: J142.1, J144.DO, U24.16
- removed net MISO24: J148.1, J150.DO, U25.16
- removed net MISO25: J154.1, J156.DO, U26.16
- removed net MISO26: J160.1, J162.DO, U27.16
- removed net MISO27: J166.1, J168.DO, U28.16
- removed net MISO8: J52.1, J54.DO, U9.16
- removed net MISO9: J58.1, J60.DO, U10.16
- removed net MOSI10: J64.4, J66.DI, U11.15
- removed net MOSI11: J70.4, J72.DI, U12.15
- removed net MOSI12: J76.4, J78.DI, U13.15
- removed net MOSI13: J82.4, J84.DI, U14.15
- removed net MOSI14: J88.4, J90.DI, U15.15
- removed net MOSI15: J94.4, J96.DI, U16.15
- removed net MOSI16: J100.4, J102.DI, U17.15
- removed net MOSI17: J106.4, J108.DI, U18.15
- removed net MOSI18: J112.4, J114.DI, U19.15
- removed net MOSI19: J118.4, J120.DI, U20.15
- removed net MOSI20: J124.4, J126.DI, U21.15
- removed net MOSI21: J130.4, J132.DI, U22.15
- removed net MOSI22: J136.4, J138.DI, U23.15
- removed net MOSI23: J142.4, J144.DI, U24.15
- removed net MOSI24: J148.4, J150.DI, U25.15
- removed net MOSI25: J154.4, J156.DI, U26.15
- removed net MOSI26: J160.4, J162.DI, U27.15
- removed net MOSI27: J166.4, J168.DI, U28.15
- removed net MOSI8: J52.4, J54.DI, U9.15
- removed net MOSI9: J58.4, J60.DI, U10.15
- removed net N$102: D30.A, R87.2
- removed net N$103: R87.1, U15.9
- removed net N$104: I2C14.1, R89.2
- removed net N$105: I2C14.3, R88.2
- removed net N$106: D31.A, R92.2
- removed net N$107: Q16.1, U16.8
- removed net N$108: Q16.3, U16.7
- removed net N$109: D32.A, R93.2
- removed net N$110: R93.1, U16.9
- removed net N$111: I2C15.1, R95.2
- removed net N$112: I2C15.3, R94.2
- removed net N$113: D33.A, R98.2
- removed net N$114: Q17.1, U17.8
- removed net N$115: Q17.3, U17.7
- removed net N$116: D34.A, R99.2
- removed net N$117: R99.1, U17.9
- removed net N$118: I2C16.1, R101.2
- removed net N$119: I2C16.3, R100.2
- removed net N$120: D35.A, R104.2
- removed net N$121: Q18.1, U18.8
- removed net N$122: Q18.3, U18.7
- removed net N$123: D36.A, R105.2
- removed net N$124: R105.1, U18.9
- removed net N$125: I2C17.1, R107.2
- removed net N$126: I2C17.3, R106.2
- removed net N$127: D37.A, R110.2
- removed net N$128: Q19.1, U19.8
- removed net N$129: Q19.3, U19.7
- removed net N$130: D38.A, R111.2
- removed net N$131: R111.1, U19.9
- removed net N$132: I2C18.1, R113.2
- removed net N$133: I2C18.3, R112.2
- removed net N$134: D39.A, R116.2
- removed net N$135: Q20.1, U20.8
- removed net N$136: Q20.3, U20.7
- removed net N$137: D40.A, R117.2
- removed net N$138: R117.1, U20.9
- removed net N$139: I2C19.1, R119.2
- removed net N$140: I2C19.3, R118.2
- removed net N$141: D41.A, R122.2
- removed net N$142: Q21.1, U21.8
- removed net N$143: Q21.3, U21.7
- removed net N$144: D42.A, R123.2
- removed net N$145: R123.1, U21.9
- removed net N$146: I2C20.1, R125.2
- removed net N$147: I2C20.3, R124.2
- removed net N$148: D43.A, R128.2
- removed net N$149: Q22.1, U22.8
- removed net N$150: Q22.3, U22.7
- removed net N$151: D44.A, R129.2
- removed net N$152: R129.1, U22.9
- removed net N$153: I2C21.1, R131.2
- removed net N$154: I2C21.3, R130.2
- removed net N$155: D45.A, R134.2
- removed net N$156: Q23.1, U23.8
- removed net N$157: Q23.3, U23.7
- removed net N$158: D46.A, R135.2
- removed net N$159: R135.1, U23.9
- removed net N$16 (its old number): Q3.1, U3.8
- removed net N$160: I2C22.1, R137.2
- removed net N$161: I2C22.3, R136.2
- removed net N$162: D47.A, R140.2
- removed net N$163: Q24.1, U24.8
- removed net N$164: Q24.3, U24.7
- removed net N$165: D48.A, R141.2
- removed net N$166: R141.1, U24.9
- removed net N$167: I2C23.1, R143.2
- removed net N$168: I2C23.3, R142.2
- removed net N$169: D49.A, R146.2
- removed net N$17 (its old number): Q3.3, U3.7
- removed net N$170: Q25.1, U25.8
- removed net N$171: Q25.3, U25.7
- removed net N$172: D50.A, R147.2
- removed net N$173: R147.1, U25.9
- removed net N$174: I2C24.1, R149.2
- removed net N$175: I2C24.3, R148.2
- removed net N$176: D51.A, R152.2
- removed net N$177: Q26.1, U26.8
- removed net N$178: Q26.3, U26.7
- removed net N$179: D52.A, R153.2
- removed net N$180: R153.1, U26.9
- removed net N$181: I2C25.1, R155.2
- removed net N$182: I2C25.3, R154.2
- removed net N$183: D53.A, R158.2
- removed net N$184: Q27.1, U27.8
- removed net N$185: Q27.3, U27.7
- removed net N$186: D54.A, R159.2
- removed net N$187: R159.1, U27.9
- removed net N$188: I2C26.1, R161.2
- removed net N$189: I2C26.3, R160.2
- removed net N$190: D55.A, R164.2
- removed net N$191: Q28.1, U28.8
- removed net N$192: Q28.3, U28.7
- removed net N$193: D56.A, R165.2
- removed net N$194: R165.1, U28.9
- removed net N$195: I2C27.1, R167.2
- removed net N$196: I2C27.3, R166.2
- removed net N$23 (its old number): Q4.1, U4.8
- removed net N$24 (its old number): Q4.3, U4.7
- removed net N$37 (its old number): Q6.1, U6.8
- removed net N$38 (its old number): Q6.3, U6.7
- removed net N$51 (its old number): Q8.1, U8.8
- removed net N$52 (its old number): Q8.3, U8.7
- removed net N$57: D17.A, R50.2
- removed net N$60: D18.A, R51.2
- removed net N$61: R51.1, U9.9
- removed net N$62: I2C8.1, R53.2
- removed net N$63: I2C8.3, R52.2
- removed net N$64: D19.A, R56.2
- removed net N$65: Q10.1, U10.8
- removed net N$66: Q10.3, U10.7
- removed net N$67: D20.A, R57.2
- removed net N$68: R57.1, U10.9
- removed net N$69: I2C9.1, R59.2
- removed net N$70: I2C9.3, R58.2
- removed net N$71: D21.A, R62.2
- removed net N$74: D22.A, R63.2
- removed net N$75: R63.1, U11.9
- removed net N$76: I2C10.1, R65.2
- removed net N$77: I2C10.3, R64.2
- removed net N$78: D23.A, R68.2
- removed net N$79: Q12.1, U12.8
- removed net N$80: Q12.3, U12.7
- removed net N$81: D24.A, R69.2
- removed net N$82: R69.1, U12.9
- removed net N$83: I2C11.1, R71.2
- removed net N$84: I2C11.3, R70.2
- removed net N$85: D25.A, R74.2
- removed net N$88: D26.A, R75.2
- removed net N$89: R75.1, U13.9
- removed net N$90: I2C12.1, R77.2
- removed net N$91: I2C12.3, R76.2
- removed net N$92: D27.A, R80.2
- removed net N$93: Q14.1, U14.8
- removed net N$94: Q14.3, U14.7
- removed net N$95: D28.A, R81.2
- removed net N$96: R81.1, U14.9
- removed net N$97: I2C13.1, R83.2
- removed net N$98: I2C13.3, R82.2
- removed net N$99: D29.A, R86.2
- removed net RST10: C32.1, J64.5, R61.1, U11.29
- removed net RST11: C35.1, J70.5, R67.1, U12.29
- removed net RST12: C38.1, J76.5, R73.1, U13.29
- removed net RST13: C41.1, J82.5, R79.1, U14.29
- removed net RST14: C44.1, J88.5, R85.1, U15.29
- removed net RST15: C47.1, J94.5, R91.1, U16.29
- removed net RST16: C50.1, J100.5, R97.1, U17.29
- removed net RST17: C53.1, J106.5, R103.1, U18.29
- removed net RST18: C56.1, J112.5, R109.1, U19.29
- removed net RST19: C59.1, J118.5, R115.1, U20.29
- removed net RST20: C62.1, J124.5, R121.1, U21.29
- removed net RST21: C65.1, J130.5, R127.1, U22.29
- removed net RST22: C68.1, J136.5, R133.1, U23.29
- removed net RST23: C71.1, J142.5, R139.1, U24.29
- removed net RST24: C74.1, J148.5, R145.1, U25.29
- removed net RST25: C77.1, J154.5, R151.1, U26.29
- removed net RST26: C80.1, J160.5, R157.1, U27.29
- removed net RST27: C83.1, J166.5, R163.1, U28.29
- removed net RST8: C26.1, J52.5, R49.1, U9.29
- removed net RST9: C29.1, J58.5, R55.1, U10.29
- removed net RXI10: J65.4, U11.30
- removed net RXI11: J71.4, U12.30
- removed net RXI12: J77.4, U13.30
- removed net RXI13: J83.4, U14.30
- removed net RXI14: J89.4, U15.30
- removed net RXI15: J95.4, U16.30
- removed net RXI16: J101.4, U17.30
- removed net RXI17: J107.4, U18.30
- removed net RXI18: J113.4, U19.30
- removed net RXI19: J119.4, U20.30
- removed net RXI20: J125.4, U21.30
- removed net RXI21: J131.4, U22.30
- removed net RXI22: J137.4, U23.30
- removed net RXI23: J143.4, U24.30
- removed net RXI24: J149.4, U25.30
- removed net RXI25: J155.4, U26.30
- removed net RXI26: J161.4, U27.30
- removed net RXI27: J167.4, U28.30
- removed net RXI8: J53.4, U9.30
- removed net RXI9: J59.4, U10.30
- removed net SCK10: J64.3, J66.SCLK, R62.1, U11.17
- removed net SCK11: J70.3, J72.SCLK, R68.1, U12.17
- removed net SCK12: J76.3, J78.SCLK, R74.1, U13.17
- removed net SCK13: J82.3, J84.SCLK, R80.1, U14.17
- removed net SCK14: J88.3, J90.SCLK, R86.1, U15.17
- removed net SCK15: J94.3, J96.SCLK, R92.1, U16.17
- removed net SCK16: J100.3, J102.SCLK, R98.1, U17.17
- removed net SCK17: J106.3, J108.SCLK, R104.1, U18.17
- removed net SCK18: J112.3, J114.SCLK, R110.1, U19.17
- removed net SCK19: J118.3, J120.SCLK, R116.1, U20.17
- removed net SCK20: J124.3, J126.SCLK, R122.1, U21.17
- removed net SCK21: J130.3, J132.SCLK, R128.1, U22.17
- removed net SCK22: J136.3, J138.SCLK, R134.1, U23.17
- removed net SCK23: J142.3, J144.SCLK, R140.1, U24.17
- removed net SCK24: J148.3, J150.SCLK, R146.1, U25.17
- removed net SCK25: J154.3, J156.SCLK, R152.1, U26.17
- removed net SCK26: J160.3, J162.SCLK, R158.1, U27.17
- removed net SCK27: J166.3, J168.SCLK, R164.1, U28.17
- removed net SCK8: J52.3, J54.SCLK, R50.1, U9.17
- removed net SCK9: J58.3, J60.SCLK, R56.1, U10.17
- removed net SCL10: J61.4, J62.4, J63.4, R64.1, U11.28
- removed net SCL11: J67.4, J68.4, J69.4, R70.1, U12.28
- removed net SCL12: J73.4, J74.4, J75.4, R76.1, U13.28
- removed net SCL13: J79.4, J80.4, J81.4, R82.1, U14.28
- removed net SCL14: J85.4, J86.4, J87.4, R88.1, U15.28
- removed net SCL15: J91.4, J92.4, J93.4, R94.1, U16.28
- removed net SCL16: J97.4, J98.4, J99.4, R100.1, U17.28
- removed net SCL17: J103.4, J104.4, J105.4, R106.1, U18.28
- removed net SCL18: J109.4, J110.4, J111.4, R112.1, U19.28
- removed net SCL19: J115.4, J116.4, J117.4, R118.1, U20.28
- removed net SCL20: J121.4, J122.4, J123.4, R124.1, U21.28
- removed net SCL21: J127.4, J128.4, J129.4, R130.1, U22.28
- removed net SCL22: J133.4, J134.4, J135.4, R136.1, U23.28
- removed net SCL23: J139.4, J140.4, J141.4, R142.1, U24.28
- removed net SCL24: J145.4, J146.4, J147.4, R148.1, U25.28
- removed net SCL25: J151.4, J152.4, J153.4, R154.1, U26.28
- removed net SCL26: J157.4, J158.4, J159.4, R160.1, U27.28
- removed net SCL27: J163.4, J164.4, J165.4, R166.1, U28.28
- removed net SCL8: J49.4, J50.4, J51.4, R52.1, U9.28
- removed net SCL9: J55.4, J56.4, J57.4, R58.1, U10.28
- removed net SDA10: J61.3, J62.3, J63.3, R65.1, U11.27
- removed net SDA11: J67.3, J68.3, J69.3, R71.1, U12.27
- removed net SDA12: J73.3, J74.3, J75.3, R77.1, U13.27
- removed net SDA13: J79.3, J80.3, J81.3, R83.1, U14.27
- removed net SDA14: J85.3, J86.3, J87.3, R89.1, U15.27
- removed net SDA15: J91.3, J92.3, J93.3, R95.1, U16.27
- removed net SDA16: J97.3, J98.3, J99.3, R101.1, U17.27
- removed net SDA17: J103.3, J104.3, J105.3, R107.1, U18.27
- removed net SDA18: J109.3, J110.3, J111.3, R113.1, U19.27
- removed net SDA19: J115.3, J116.3, J117.3, R119.1, U20.27
- removed net SDA20: J121.3, J122.3, J123.3, R125.1, U21.27
- removed net SDA21: J127.3, J128.3, J129.3, R131.1, U22.27
- removed net SDA22: J133.3, J134.3, J135.3, R137.1, U23.27
- removed net SDA23: J139.3, J140.3, J141.3, R143.1, U24.27
- removed net SDA24: J145.3, J146.3, J147.3, R149.1, U25.27
- removed net SDA25: J151.3, J152.3, J153.3, R155.1, U26.27
- removed net SDA26: J157.3, J158.3, J159.3, R161.1, U27.27
- removed net SDA27: J163.3, J164.3, J165.3, R167.1, U28.27
- removed net SDA8: J49.3, J50.3, J51.3, R53.1, U9.27
- removed net SDA9: J55.3, J56.3, J57.3, R59.1, U10.27
- removed net TXO10: J65.5, U11.31
- removed net TXO11: J71.5, U12.31
- removed net TXO12: J77.5, U13.31
- removed net TXO13: J83.5, U14.31
- removed net TXO14: J89.5, U15.31
- removed net TXO15: J95.5, U16.31
- removed net TXO16: J101.5, U17.31
- removed net TXO17: J107.5, U18.31
- removed net TXO18: J113.5, U19.31
- removed net TXO19: J119.5, U20.31
- removed net TXO20: J125.5, U21.31
- removed net TXO21: J131.5, U22.31
- removed net TXO22: J137.5, U23.31
- removed net TXO23: J143.5, U24.31
- removed net TXO24: J149.5, U25.31
- removed net TXO25: J155.5, U26.31
- removed net TXO26: J161.5, U27.31
- removed net TXO27: J167.5, U28.31
- removed net TXO8: J53.5, U9.31
- removed net TXO9: J59.5, U10.31
- new net !RST: R10.1, U3.2
- new net !RST1: R17.1, U4.2
- new net !RST2: R27.1, U6.2
- new net !RST3: R37.1, U8.2
- new net !RST4: R47.1, U10.2
- new net !RST5: R57.1, U12.2
- new net !RST6: R67.1, U14.2
- new net !RST7: R77.1, U16.2
- new net VBACKUP: C2.1, R7.1, U3.6
- new net VBACKUP1: C7.1, R18.1, U4.6
- new net VBACKUP2: C11.1, R28.1, U6.6
- new net VBACKUP3: C15.1, R38.1, U8.6
- new net VBACKUP4: C19.1, R48.1, U10.6
- new net VBACKUP5: C23.1, R58.1, U12.6
- new net VBACKUP6: C27.1, R68.1, U14.6
- new net VBACKUP7: C31.1, R78.1, U16.6
- new net V_BATT: BT1.+, R10.2, R7.2
- new net V_BATT1: BT2.+, R17.2, R18.2
- new net V_BATT2: BT3.+, R27.2, R28.2
- new net V_BATT3: BT4.+, R37.2, R38.2
- new net V_BATT4: BT5.+, R47.2, R48.2
- new net V_BATT5: BT6.+, R57.2, R58.2
- new net V_BATT6: BT7.+, R67.2, R68.2
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Routing:
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- removed copper zone on layer 1, net GND10
- removed copper zone on layer 16, net GND10
- removed copper zone on layer 1, net GND11
- removed copper zone on layer 16, net GND11
- removed copper zone on layer 1, net GND12
- removed copper zone on layer 16, net GND12
- removed copper zone on layer 1, net GND13
- removed copper zone on layer 16, net GND13
- removed copper zone on layer 1, net GND14
- removed copper zone on layer 16, net GND14
- removed copper zone on layer 1, net GND15
- removed copper zone on layer 16, net GND15
- removed copper zone on layer 1, net GND16
- removed copper zone on layer 16, net GND16
- removed copper zone on layer 1, net GND17
- removed copper zone on layer 16, net GND17
- removed copper zone on layer 1, net GND18
- removed copper zone on layer 16, net GND18
- removed copper zone on layer 1, net GND19
- removed copper zone on layer 16, net GND19
- removed copper zone on layer 1, net GND20
- removed copper zone on layer 16, net GND20
- removed copper zone on layer 1, net GND21
- removed copper zone on layer 16, net GND21
- removed copper zone on layer 1, net GND22
- removed copper zone on layer 16, net GND22
- removed copper zone on layer 1, net GND23
- removed copper zone on layer 16, net GND23
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Other:
- board size 200.9 x 128.3 mm -> 96.8 x 174 mm
- board text added: "Units in Inches"
- board text added: "v10"
- board text removed: "v12"
